File: bench1/bm2.routed.kicad_pcb (KiCad board)
At the start: 2 copper layers, 50.8 x 22.9 mm, 18 parts, among them IC1 PCF8523T, SW1 KMR2, X4 microsd, Y1 32khz

Commit message: prepare to change obstacles logic
Routing:
- net GND: track 0.00 -> 55.2 mm, vias 0 -> 2
- net +3V3: track 0.00 -> 36.9 mm, vias 0 -> 5
- net SDA: track 0.00 -> 18.7 mm
- net SCL: track 0.00 -> 16.7 mm, vias 0 -> 2
- net RESET: track 0.00 -> 16.6 mm, vias 0 -> 1
- net SCK: track 0.00 -> 13.4 mm, vias 0 -> 1
- net SD_CS: track 0.00 -> 13.0 mm, vias 0 -> 2
- net MOSI: track 0.00 -> 11.8 mm, vias 0 -> 1
- net MISO: track 0.00 -> 7.42 mm
- net INT1: track 0.00 -> 7.42 mm, vias 0 -> 1
- net N$1: track 0.00 -> 4.92 mm, vias 0 -> 4
- net CR1220: track 0.00 -> 4.27 mm
- net N$7: track 0.00 -> 4.21 mm
- net N$8: track 0.00 -> 2.53 mm
- net CS: track 0.00 -> 0.75 mm
